File: digitalphoenix_toolstick_hardware.kicad_pcb (KiCad board)
At the start: 2 copper layers, 43 parts, among them J1 USB_A, J2 Conn_01x06, J3 Conn_01x04, SW1 SW_SPST, SW2 SW_SPST, U1 AMS1117-3.3, U2 ESP32-S2, U3 W25Q128JVS, X1 40MHz 10ppm

Commit message: More PCB work
Parts:
- moved C1 89.0 mm to (63.5, 79.3), turned to 90 degrees
- moved C2 80.0 mm to (78.5, 67.6), turned to 180 degrees
- moved C3 76.3 mm to (79.0, 78.0), turned to 180 degrees
- moved C7 71.6 mm to (86.1, 75.9), turned to 270 degrees
- moved C9 71.4 mm to (81.0, 78.0), turned to 180 degrees
- moved X1 69.3 mm to (82.0, 80.4)
- moved C8 69.1 mm to (86.4, 79.8)
- moved C4 68.5 mm to (79.2, 80.5), turned to 90 degrees
- moved C6 68.4 mm to (82.5, 67.6)
- moved C5 67.8 mm to (84.6, 80.0), turned to 270 degrees
- moved C14 67.7 mm to (87.1, 74.7), turned to 270 degrees
- moved C11 67.7 mm to (87.6, 78.2), turned to 180 degrees
- moved C12 62.0 mm to (87.6, 77.2), turned to 180 degrees
- moved C10 60.0 mm to (85.1, 77.5)
- moved C13 54.8 mm to (87.6, 76.2), turned to 180 degrees
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Connections:
- U2 pad 10: Net-(U2-Pad10) -> (no net)
- U2 pad 11: Net-(U2-Pad11) -> (no net)
- U2 pad 12: Net-(U2-Pad12) -> (no net)
- U2 pad 13: Net-(U2-Pad13) -> (no net)
- U2 pad 14: Net-(U2-Pad14) -> (no net)
- U2 pad 15: Net-(U2-Pad15) -> (no net)
- U2 pad 16: Net-(U2-Pad16) -> (no net)
- U2 pad 17: Net-(U2-Pad17) -> (no net)
- U2 pad 18: Net-(U2-Pad18) -> (no net)
- U2 pad 19: Net-(U2-Pad19) -> (no net)
- U2 pad 21: Net-(U2-Pad21) -> (no net)
- U2 pad 22: Net-(U2-Pad22) -> (no net)
- U2 pad 23: Net-(U2-Pad23) -> (no net)
- U2 pad 28: Net-(U2-Pad28) -> (no net)
- U2 pad 29: Net-(U2-Pad29) -> (no net)
- U2 pad 37: Net-(U2-Pad37) -> (no net)
- U2 pad 38: Net-(U2-Pad38) -> (no net)
- U2 pad 40: Net-(U2-Pad40) -> (no net)
- U2 pad 41: Net-(U2-Pad41) -> (no net)
- U2 pad 42: Net-(U2-Pad42) -> (no net)
- U2 pad 50: Net-(U2-Pad50) -> (no net)
- U2 pad 55: Net-(U2-Pad55) -> (no net)
- U2 pad 6: Net-(U2-Pad6) -> (no net)
- U2 pad 7: Net-(U2-Pad7) -> (no net)
- U2 pad 8: Net-(U2-Pad8) -> (no net)
- U2 pad 9: Net-(U2-Pad9) -> (no net)
- X1 pad 1: Net-(C5-Pad1) -> Net-(C4-Pad1)
- X1 pad 2: Net-(C4-Pad1) -> GND
- X1 pad 3: (no net) -> Net-(C5-Pad1)
- X1 pad 4: (no net) -> GND
Routing:
- net VDD: track 0.00 -> 26.6 mm
- net +5V: track 0.00 -> 11.2 mm
- net Net-(C4-Pad1): track 0.00 -> 8.48 mm
- net VDDF: track 0.00 -> 3.73 mm
- net Net-(C5-Pad1): track 0.00 -> 3.11 mm
- net Net-(R1-Pad1): track 0.00 -> 1.85 mm
Other:
- net class Default: trace_width 0.25 -> 0.127; via_dia 0.8 -> 0.4; via_drill 0.4 -> 0.2
- rule trace_min: 0.2 -> 0.127
- rule via_min_drill: 0.3 -> 0.2
